File: NerdFlare25.kicad_pcb (KiCad board)
At the start: 2 copper layers, 110.3 x 136.7 mm, 31 parts, among them J1 VEXT, SW1 SW_Push, SW2 SW_SPDT, T1 DMG2305

Commit message: Moved some silk labels around.
Parts:
- moved R5 0.40 mm to (73.2, 79.4)
Changed lines of the file:
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@@
 		(at 91.49 80.78 3.5)
 		(property "Reference" "D5"
-			(at 0 -2.1 -176.5)
+			(at -3.466153 0.158692 3.5)
 			(unlocked yes)
 			(layer "B.SilkS")
@@
 		(tags "AA battery cell holder")
 		(property "Reference" "BT1"
-			(at -3.51514 7.44835 360)
+			(at -4.01 2.99 360)
 			(layer "B.SilkS")
 			(effects
@@
 		(tags "SOT TO_SOT_SMD")
 		(property "Reference" "T1"
-			(at 0.06713 -2.89764 360)
+			(at 2.5925 0.02 360)
 			(layer "B.SilkS")
 			(effects
@@
 		(at 104.8 80.16 1.5)
 		(property "Reference" "D6"
-			(at 0 -2.1 -178.5)
+			(at -3.403023 0.070944 1.5)
 			(unlocked yes)
 			(layer "B.SilkS")
@@
 		(tags "Through hole pin header THT 2x20 2.54mm double row")
 		(property "Reference" "A1"
-			(at 6.35 -27.575 360)
+			(at -0.04 0.06 360)
 			(layer "B.SilkS")
 			(effects
@@
 			(layer "B.CrtYd")
 		)
-		(fp_text user "Copper Keepouts shown on Dwgs layer"
-			(at 0.1 30.2 360)
-			(layer "Cmts.User")
-			(effects
-				(font
-					(size 1 1)
-					(thickness 0.15)
-				)
-			)
-		)
 		(fp_text user "${REFERENCE}"
 			(at 0 0 360)
@@
 		(tags "resistor handsolder")
 		(property "Reference" "R10"
-			(at 0 1.82 90)
+			(at -4.19 0.03 -90)
 			(layer "B.SilkS")
 			(effects
@@
 		(tags "resistor handsolder")
 		(property "Reference" "R8"
-			(at 0 1.82 360)
+			(at 0.04 -1.77 360)
 			(layer "B.SilkS")
 			(effects
@@
 		(tags "resistor handsolder")
 		(property "Reference" "R3"
-			(at 0 1.82 0)
+			(at 0.02 -2.03 0)
 			(layer "B.SilkS")
 			(effects
@@
 		(tags "AA battery cell holder")
 		(property "Reference" "BT2"
-			(at -3.51514 7.44835 360)
+			(at -3.49 -0.04 360)
 			(layer "B.SilkS")
 			(effects
@@
 		(at 134.543654 80.565365 -4)
 		(property "Reference" "D8"
-			(at 0 -2.100002 176)
+			(at -3.379761 0.030469 -4)
 			(unlocked yes)
 			(layer "B.SilkS")
@@
 		(at 117.16 80.01)
 		(property "Reference" "D7"
-			(at 0 -2.1 180)
+			(at -3.48 0.03 0)
 			(unlocked yes)
 			(layer "B.SilkS")
@@
 		(tags "resistor handsolder")
 		(property "Reference" "R6"
-			(at 0 1.82 360)
+			(at 0.11 -1.75 360)
 			(layer "B.SilkS")
 			(effects
@@
 		(at 73.308217 82.206793 6)
 		(property "Reference" "D4"
-			(at 0 -2.1 -174)
+			(at -3.391912 0.048924 6)
 			(unlocked yes)
 			(layer "B.SilkS")
@@
 		(tags "resistor handsolder")
 		(property "Reference" "R1"
-			(at 0 1.82 0)
+			(at -3.65 0.03 0)
 			(layer "B.SilkS")
 			(effects
@@
 		(at 106.81 103.58 180)
 		(property "Reference" "D1"
-			(at 0 -2.1 0)
+			(at -3.4 -0.19 0)
 			(unlocked yes)
 			(layer "B.SilkS")
@@
 		(tags "resistor handsolder")
 		(property "Reference" "R9"
-			(at 0 1.82 360)
+			(at 0.03 -1.73 360)
 			(layer "B.SilkS")
 			(effects
@@
 		(tags "resistor handsolder")
 		(property "Reference" "R2"
-			(at 0 1.82 360)
+			(at 0.06 -1.63 360)
 			(layer "B.SilkS")
 			(effects
@@
 		)
 		(property "Value" "680"
-			(at 0 -1.82 360)
-			(layer "B.Fab")
+			(at 0.01 1.89 0)
+			(layer "B.SilkS")
 			(effects
 				(font
@@
 	(footprint "Resistor_SMD:R_1206_3216Metric_Pad1.30x1.75mm_HandSolder"
 		(layer "B.Cu")
-		(at 73.24 79.79)
+		(at 73.16 79.4)
 		(descr "Resistor SMD 1206 (3216 Metric), square (rectangular) end terminal, IPC_7351 nominal with elongated pad for handsoldering. (Body size source: IPC-SM-782 page 72, https://www.pcb-3d.com/wordpress/wp-content/uploads/ipc-sm-782a_amendment_1_and_2.pdf), generated with kicad-footprint-generator")
 		(tags "resistor handsolder")
 		(property "Reference" "R5"
-			(at 0 1.82 360)
+			(at -0.08 -1.86 360)
 			(layer "B.SilkS")
 			(effects
@@
 		(tags "resistor handsolder")
 		(property "Reference" "R7"
-			(at 0 1.82 360)
+			(at 0.08 -1.73 360)
 			(layer "B.SilkS")
 			(effects
@@
 	)
 	(zone
-		(net 0)
-		(net_name "")
-		(layer "F.Cu")
-		(hatch edge 0.5)
-		(connect_pads
-			(clearance 0)
-		)
-		(min_thickness 0.25)
-		(filled_areas_thickness no)
-		(keepout
-			(tracks not_allowed)
-			(vias not_allowed)
-			(pads not_allowed)
-			(copperpour not_allowed)
-			(footprints not_allowed)
-		)
-		(fill
-			(thermal_gap 0.5)
-			(thermal_bridge_width 0.5)
-		)
-		(polygon
-			(pts
-				(xy 134.81 111.39) (xy 135.82 111.5) (xy 136.39 113.08) (xy 135.49 114.06) (xy 133.91 113.95) (xy 133.32 112.66)
-				(xy 133.99 111.53)
-			)
-		)
-	)
-	(zone

Commit message: This is v0; going to fab.
Parts:
- removed J1: VEXT, nerdflare25:SAO_PinHeader_1x02_P2.54mm_SMD
- removed JP1: SolderJumper_3_Open, nerdflare25:SolderJumper_Open_Rounded_SAO
- removed LED1: LED, LED_SMD:LED_0805_2012Metric_Pad1.15x1.40mm_HandSolder
- removed the R2 at (121.4, 111.6)
- removed S1: SW_Slide_SPDT, nerdflare25:SW_Slide-03_Wuerth-WS-SLTV_10x2.5x6.4_P2.54mm
- added D11: LED, LED_SMD:LED_0805_2012Metric_Pad1.15x1.40mm_HandSolder, B.Cu at (145.7, 154.5)
- added R11: 680, Resistor_SMD:R_1206_3216Metric_Pad1.30x1.75mm_HandSolder, B.Cu at (145.7, 149.7)
- added R12: 100, Resistor_SMD:R_1206_3216Metric_Pad1.30x1.75mm_HandSolder, B.Cu at (72.3, 142.0)
- SW2: moved to B.Cu
- moved SW2 198.2 mm to (164.5, 119.3), turned to -90 degrees
- moved T1 21.8 mm to (146.8, 158.7), turned to 0 degrees
- moved D4 0.64 mm to (65.0, 100.2)
- moved D1 0.60 mm to (136.2, 102.0)
- moved R1 0.60 mm to (141.6, 101.2)
- moved D2 0.58 mm to (106.9, 104.2)
- moved R2 0.58 mm to (106.8, 106.8)
- moved D6 0.57 mm to (91.5, 80.2)
- moved R6 0.57 mm to (91.5, 77.7), turned to 180 degrees
- moved D5 0.50 mm to (73.3, 81.7)
- moved R5 0.50 mm to (73.2, 78.9), turned to 180 degrees
- moved R3 0.48 mm to (85.7, 107.7), turned to 0 degrees
- moved D3 0.48 mm to (80.5, 107.4)
- moved R7 0.43 mm to (160.6, 88.6), turned to 90 degrees
- moved D10 0.38 mm to (104.8, 79.8)
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- renumbered D10 to D1, D6 to D10, D1 to D2, D2 to D3, D3 to D4, D4 to D5, D5 to D6, D9 to D7, D7 to D9, R11 to R1, R7 to R10, R1 to R2, R10 to R7, R9 to R8, R8 to R9
Connections:
- A1 pad 11: /SW1 -> Net-(A1-GP8)
- A1 pad 15: unconnected-(A1-GP11-Pad15) -> Net-(A1-GP11)
- A1 pad 16: unconnected-(A1-GP12-Pad16) -> Net-(A1-GP12)
- A1 pad 17: unconnected-(A1-GP13-Pad17) -> Net-(A1-GP13)
- A1 pad 19: unconnected-(A1-GP14-Pad19) -> Net-(A1-GP14)
- A1 pad 20: unconnected-(A1-GP15-Pad20) -> Net-(A1-GP15)
- A1 pad 21: unconnected-(A1-GP16-Pad21) -> Net-(A1-GP16)
- A1 pad 22: unconnected-(A1-GP17-Pad22) -> Net-(A1-GP17)
- A1 pad 24: unconnected-(A1-GP18-Pad24) -> Net-(A1-GP18)
- A1 pad 25: unconnected-(A1-GP19-Pad25) -> Net-(A1-GP19)
- A1 pad 26: unconnected-(A1-GP20-Pad26) -> Net-(A1-GP20)
- A1 pad 36: Net-(A1-3V3_OUT) -> unconnected-(A1-3V3_OUT-Pad36)
- D1 pad 2: unconnected-(D10-A-Pad2) -> Net-(A1-GP16)
- D10 pad 2: unconnected-(D6-A-Pad2) -> Net-(A1-GP20)
- D2 pad 2: unconnected-(D1-A-Pad2) -> Net-(A1-GP15)
- D3 pad 2: unconnected-(D2-A-Pad2) -> Net-(A1-GP14)
- D4 pad 2: unconnected-(D3-A-Pad2) -> Net-(A1-GP13)
- D5 pad 2: unconnected-(D4-A-Pad2) -> Net-(A1-GP12)
- D6 pad 2: unconnected-(D5-A-Pad2) -> Net-(A1-GP11)
- D7 pad 2: unconnected-(D9-A-Pad2) -> Net-(A1-GP17)
- D8 pad 2: unconnected-(D8-A-Pad2) -> Net-(A1-GP18)
- D9 pad 2: unconnected-(D7-A-Pad2) -> Net-(A1-GP19)
- R1 pad 2: unconnected-(R11-Pad2) -> GND
- R10 pad 2: unconnected-(R7-Pad2) -> GND
- R2 pad 2: unconnected-(R1-Pad2) -> GND
- R3 pad 2: unconnected-(R3-Pad2) -> GND
- R4 pad 2: unconnected-(R4-Pad2) -> GND
- R5 pad 2: unconnected-(R5-Pad2) -> GND
- R6 pad 2: unconnected-(R6-Pad2) -> GND
- R7 pad 2: unconnected-(R10-Pad2) -> GND
- R8 pad 2: unconnected-(R9-Pad2) -> GND
- R9 pad 2: unconnected-(R8-Pad2) -> GND
- SW2 pad 1: unconnected-(SW2-A-Pad1) -> Net-(BT2-+)
- SW2 pad 2: unconnected-(SW2-B-Pad2) -> Net-(SW2-B)
- SW2 pad 3: unconnected-(SW2-C-Pad3) -> GND
- T1 pad 3: Net-(JP1-A) -> Net-(SW2-B)
Routing:
- net Net-(A1-GP20): track 0.00 -> 141.7 mm
- net Net-(A1-GP19): track 0.00 -> 126.9 mm
- net Net-(A1-GP11): track 0.00 -> 113.6 mm
- net Net-(A1-GP18): track 0.00 -> 102.0 mm
- net Net-(A1-GP12): track 0.00 -> 92.5 mm
- net VDD: track 80.1 -> 0.00 mm
- net Net-(BT2-+): track 21.7 -> 85.8 mm
- net Net-(J1-Pin_1): track 61.9 -> 0.00 mm
- net Net-(A1-GP17): track 0.00 -> 60.1 mm
- net Net-(A1-GP13): track 0.00 -> 57.1 mm
- net Net-(A1-GP15): track 0.00 -> 53.2 mm
- net Net-(A1-VBUS): track 75.9 -> 27.0 mm
- net Net-(SW2-B): track 0.00 -> 47.7 mm
- net /SW1: track 43.2 -> 11.8 mm
- net Net-(A1-GP8): track 0.00 -> 30.5 mm
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Other:
- board text added: "NerdFlare Badge 2025 v0"

Commit message: This is v1 sent to production at JLCPCB; removed status LED, determined final LED colors; added silkscreen sigantures.
Parts:
- removed D11: LED, LED_SMD:LED_0805_2012Metric_Pad1.15x1.40mm_HandSolder
- removed R11: 680, Resistor_SMD:R_1206_3216Metric_Pad1.30x1.75mm_HandSolder
- added G***: LOGO, LOGO, B.Cu at (152.3, 64.6)
- Pico W/2 W: renamed from A1
- R1, R10, R2, R3, R4, R5, R6, R7, R8, R9: value R -> 65R
- moved T1 18.8 mm to (147.8, 139.9), turned to 90 degrees
Routing:
- net Net-(SW2-B): track 47.7 -> 26.9 mm
- net Net-(A1-VBUS): track 27.0 -> 46.3 mm
- net Net-(A1-VSYS): track 26.8 -> 41.5 mm
- net Net-(A1-GP13): track 57.1 -> 63.6 mm
- net Net-(A1-GP11): track 113.6 -> 116.9 mm
- net Net-(A1-GP12): track 92.5 -> 95.8 mm
- net Net-(D11-K): track 2.22 -> 0.00 mm
Other:
- board text added: "2025"
- board text added: "@Hankashyyyk"
- board text added: "Flare"
- board text added: "Nerd"
- board text added: "NerdFlare Badge 2025 v1"
- board text added: "cal poly"
- board text added: "mode"
- board text added: "on off"
- board text added: "znjp"
- board text removed: "NerdFlare Badge 2025 v0"

Commit message: v1.1 flipped on the on/off switch label loll
Other:
- board text added: "NerdFlare Badge 2025 v1.1"
- board text added: "off on"
- board text removed: "NerdFlare Badge 2025 v1"
- board text removed: "on off"
Changed lines of the file:
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@@
 		)
 	)
-	(gr_text "NerdFlare Badge 2025 v1"
+	(gr_text "NerdFlare Badge 2025 v1.1"
 		(at 121.64 170.89 0)
 		(layer "B.SilkS")
@@
 		)
 	)
-	(gr_text "on   off"
+	(gr_text "off   on"
 		(at 159.207542 123.293986 270)
 		(layer "B.SilkS")
@@
 			(justify left bottom mirror)
 		)
-		(render_cache "on   off" 270
+		(render_cache "off   on" 270
 			(polygon
 				(pts
@@
 			(polygon
 				(pts
-					(xy 161.3608 121.200336) (xy 161.196669 121.209617) (xy 161.277527 121.147035) (xy 161.340114 121.067503)
-					(xy 161.343215 121.062094) (xy 161.379851 120.968061) (xy 161.392016 120.867926) (xy 161.392063 120.860838)
-					(xy 161.382652 120.760912) (xy 161.347884 120.663086) (xy 161.325141 120.627342) (xy 161.25478 120.556438)
-					(xy 161.16293 120.512276) (xy 161.156613 120.510594) (xy 161.051567 120.493515) (xy 160.952489 120.486792)
-					(xy 160.84632 120.484319) (xy 160.817116 120.484216) (xy 159.547542 120.484216) (xy 159.547542 121.039136)
-					(xy 160.808812 121.039136) (xy 160.911995 121.040376) (xy 161.012924 121.046887) (xy 161.037911 121.051836)
-					(xy 161.079433 121.120224) (xy 161.03205 121.194474) (xy 160.928666 121.206719) (xy 160.827954 121.20938)
-					(xy 160.779014 121.209617) (xy 159.547542 121.209617) (xy 159.547542 121.764537) (xy 161.3608 121.764537)
+					(xy 161.76722 121.05721) (xy 161.485853 121.05721) (xy 161.484063 121.158521) (xy 161.471641 121.25784)
+					(xy 161.47071 121.259931) (xy 161.384736 121.290706) (xy 161.329537 121.290706) (xy 161.329537 121.05721)
+					(xy 161.04817 121.05721) (xy 161.04817 121.189101) (xy 159.547542 121.189101) (xy 159.547542 121.74402)
+					(xy 161.04817 121.74402) (xy 161.04817 121.858326) (xy 161.329537 121.858326) (xy 161.329537 121.74402)
+					(xy 161.428608 121.742828) (xy 161.528839 121.737151) (xy 161.565964 121.731808) (xy 161.6541 121.687629)
+					(xy 161.671966 121.670748) (xy 161.725384 121.58511) (xy 161.742796 121.533972) (xy 161.760327 121.430073)
+					(xy 161.766362 121.326594) (xy 161.76722 121.26042)
 				)
 			)
 			(polygon
 				(pts
-					(xy 160.803129 117.56973) (xy 160.908875 117.576945) (xy 161.010068 117.595311) (xy 161.015954 117.597035)
-					(xy 161.108583 117.636816) (xy 161.192761 117.694962) (xy 161.230044 117.729727) (xy 161.290726 117.809795)
-					(xy 161.336865 117.901592) (xy 161.343549 117.918531) (xy 161.372604 118.019129) (xy 161.387697 118.121501)
-					(xy 161.392063 118.222527) (xy 161.389965 118.290052) (xy 161.377874 118.390054) (xy 161.351428 118.490732)
-					(xy 161.30609 118.587914) (xy 161.246871 118.668524) (xy 161.169057 118.73747) (xy 161.077967 118.785751)
-					(xy 161.000237 118.809687) (xy 160.896295 118.82844) (xy 160.789241 118.837843) (xy 160.684248 118.840461)
-					(xy 160.220186 118.840461) (xy 160.177969 118.840195) (xy 160.075295 118.836883) (xy 159.977012 118.828631)
-					(xy 159.874338 118.810175) (xy 159.853023 118.804145) (xy 159.761501 118.766691) (xy 159.677967 118.709547)
-					(xy 159.653617 118.686029) (xy 159.595968 118.60546) (xy 159.556334 118.511222) (xy 159.551484 118.495005)
-					(xy 159.5304 118.397964) (xy 159.519447 118.298226) (xy 159.51645 118.204453) (xy 159.828909 118.204453)
-					(xy 159.867988 118.268933) (xy 159.935533 118.281892) (xy 160.037493 118.285542) (xy 160.865476 118.285542)
-					(xy 160.943242 118.28392) (xy 161.042796 118.268933) (xy 161.079433 118.202988) (xy 161.042796 118.138507)
-					(xy 160.968659 118.126263) (xy 160.865476 118.123364) (xy 160.019419 118.123364) (xy 159.965227 118.124372)
-					(xy 159.864569 118.139484) (xy 159.828909 118.204453) (xy 159.51645 118.204453) (xy 159.516278 118.19908)
-					(xy 159.519988 118.10922) (xy 159.534597 118.007578) (xy 159.563173 117.906965) (xy 159.582745 117.860952)
-					(xy 159.637523 117.772333) (xy 159.70923 117.69887) (xy 159.740576 117.674914) (xy 159.825425 117.625575)
-					(xy 159.92221 117.593357) (xy 159.978246 117.58365) (xy 160.07995 117.573919) (xy 160.179655 117.569637)
-					(xy 160.28027 117.568445) (xy 160.723815 117.568445)
+					(xy 161.76722 120.248277) (xy 161.485853 120.248277) (xy 161.484063 120.349589) (xy 161.471641 120.448908)
+					(xy 161.47071 120.450999) (xy 161.384736 120.481773) (xy 161.329537 120.481773) (xy 161.329537 120.248277)
+					(xy 161.04817 120.248277) (xy 161.04817 120.380168) (xy 159.547542 120.380168) (xy 159.547542 120.935088)
+					(xy 161.04817 120.935088) (xy 161.04817 121.049394) (xy 161.329537 121.049394) (xy 161.329537 120.935088)
+					(xy 161.428608 120.933895) (xy 161.528839 120.928219) (xy 161.565964 120.922876) (xy 161.6541 120.878697)
+					(xy 161.671966 120.861815) (xy 161.725384 120.776178) (xy 161.742796 120.725039) (xy 161.760327 120.621141)
+					(xy 161.766362 120.517662) (xy 161.76722 120.451487)
 				)
 			)
 			(polygon
 				(pts
-					(xy 161.76722 116.68624) (xy 161.485853 116.68624) (xy 161.484063 116.787551) (xy 161.471641 116.88687)
-					(xy 161.47071 116.888961) (xy 161.384736 116.919736) (xy 161.329537 116.919736) (xy 161.329537 116.68624)
-					(xy 161.04817 116.68624) (xy 161.04817 116.818131) (xy 159.547542 116.818131) (xy 159.547542 117.37305)
-					(xy 161.04817 117.37305) (xy 161.04817 117.487356) (xy 161.329537 117.487356) (xy 161.329537 117.37305)
-					(xy 161.428608 117.371858) (xy 161.528839 117.366181) (xy 161.565964 117.360838) (xy 161.6541 117.316659)
-					(xy 161.671966 117.299778) (xy 161.725384 117.21414) (xy 161.742796 117.163002) (xy 161.760327 117.059103)
-					(xy 161.766362 116.955624) (xy 161.76722 116.88945)
+					(xy 160.803129 117.415369) (xy 160.908875 117.422584) (xy 161.010068 117.44095) (xy 161.015954 117.442674)
+					(xy 161.108583 117.482455) (xy 161.192761 117.540601) (xy 161.230044 117.575366) (xy 161.290726 117.655433)
+					(xy 161.336865 117.74723) (xy 161.343549 117.764169) (xy 161.372604 117.864767) (xy 161.387697 117.967139)
+					(xy 161.392063 118.068166) (xy 161.389965 118.13569) (xy 161.377874 118.235692) (xy 161.351428 118.336371)
+					(xy 161.30609 118.433553) (xy 161.246871 118.514163) (xy 161.169057 118.583108) (xy 161.077967 118.63139)
+					(xy 161.000237 118.655325) (xy 160.896295 118.674079) (xy 160.789241 118.683482) (xy 160.684248 118.6861)
+					(xy 160.220186 118.6861) (xy 160.177969 118.685834) (xy 160.075295 118.682521) (xy 159.977012 118.674269)
+					(xy 159.874338 118.655814) (xy 159.853023 118.649783) (xy 159.761501 118.61233) (xy 159.677967 118.555186)
+					(xy 159.653617 118.531668) (xy 159.595968 118.451098) (xy 159.556334 118.356861) (xy 159.551484 118.340643)
+					(xy 159.5304 118.243603) (xy 159.519447 118.143864) (xy 159.51645 118.050092) (xy 159.828909 118.050092)
+					(xy 159.867988 118.114572) (xy 159.935533 118.127531) (xy 160.037493 118.13118) (xy 160.865476 118.13118)
+					(xy 160.943242 118.129558) (xy 161.042796 118.114572) (xy 161.079433 118.048626) (xy 161.042796 117.984146)
+					(xy 160.968659 117.971901) (xy 160.865476 117.969003) (xy 160.019419 117.969003) (xy 159.965227 117.97001)
+					(xy 159.864569 117.985123) (xy 159.828909 118.050092) (xy 159.51645 118.050092) (xy 159.516278 118.044718)
+					(xy 159.519988 117.954859) (xy 159.534597 117.853217) (xy 159.563173 117.752604) (xy 159.582745 117.706591)
+					(xy 159.637523 117.617972) (xy 159.70923 117.544509) (xy 159.740576 117.520552) (xy 159.825425 117.471213)
+					(xy 159.92221 117.438996) (xy 159.978246 117.429289) (xy 160.07995 117.419557) (xy 160.179655 117.415275)
+					(xy 160.28027 117.414083) (xy 160.723815 117.414083)
 				)
 			)
 			(polygon
 				(pts
-					(xy 161.76722 115.877307) (xy 161.485853 115.877307) (xy 161.484063 115.978619) (xy 161.471641 116.077938)
-					(xy 161.47071 116.080029) (xy 161.384736 116.110803) (xy 161.329537 116.110803) (xy 161.329537 115.877307)
-					(xy 161.04817 115.877307) (xy 161.04817 116.009198) (xy 159.547542 116.009198) (xy 159.547542 116.564118)
-					(xy 161.04817 116.564118) (xy 161.04817 116.678424) (xy 161.329537 116.678424) (xy 161.329537 116.564118)
-					(xy 161.428608 116.562925) (xy 161.528839 116.557249) (xy 161.565964 116.551906) (xy 161.6541 116.507727)
-					(xy 161.671966 116.490845) (xy 161.725384 116.405208) (xy 161.742796 116.354069) (xy 161.760327 116.250171)
-					(xy 161.766362 116.146692) (xy 161.76722 116.080517)
+					(xy 161.3608 116.675004) (xy 161.196669 116.684286) (xy 161.277527 116.621703) (xy 161.340114 116.542172)
+					(xy 161.343215 116.536763) (xy 161.379851 116.442729) (xy 161.392016 116.342595) (xy 161.392063 116.335507)
+					(xy 161.382652 116.235581) (xy 161.347884 116.137754) (xy 161.325141 116.102011) (xy 161.25478 116.031106)
+					(xy 161.16293 115.986944) (xy 161.156613 115.985263) (xy 161.051567 115.968184) (xy 160.952489 115.96146)
+					(xy 160.84632 115.958987) (xy 160.817116 115.958884) (xy 159.547542 115.958884) (xy 159.547542 116.513804)
+					(xy 160.808812 116.513804) (xy 160.911995 116.515044) (xy 161.012924 116.521556) (xy 161.037911 116.526505)
+					(xy 161.079433 116.594893) (xy 161.03205 116.669143) (xy 160.928666 116.681387) (xy 160.827954 116.684049)
+					(xy 160.779014 116.684286) (xy 159.547542 116.684286) (xy 159.547542 117.239205) (xy 161.3608 117.239205)
 				)
 			)
